Commit message: Vaccum gripper with interface plate visible.

File: mrk_robot_support/urdf/ur5_gripper.xacro (robot description, xacro)
@@ -1,4 +1,5 @@
 <?xml version="1.0" ?>
 <robot name="ur5_gripper" xmlns:xacro="https://ros.org/wiki/xacro">
+  <!-- start: including -->
   <!-- vacum gripper -->
   <xacro:include filename="$(find mrk_robot_support)/urdf/vacuum_gripper_macro.xacro"/>
@@ -8,11 +9,18 @@
   <!-- ur5 -->
   <xacro:include filename="$(find ur_description)/urdf/ur5.urdf.xacro" />
-  <!-- arm -->
+  <!-- end: including -->
+  <!-- start: properties -->
+  <xacro:property name="stand_radius" value="0.08" />
+  <xacro:property name="stand_length" value="0.5" />
+  <xacro:property name="stand_mass" value="20.0" />
+  <xacro:property name="arm_prefix" value=""/>
+  <!-- end: properties -->
+  <!-- start: compentens instantiating -->
+  <!-- arm instance-->
   <xacro:ur5_robot prefix="" joint_limited="true"/>
-  <!-- properties -->
-  <xacro:property name="base_radius" value="0.08" />
-  <xacro:property name="base_length" value="0.5" />
-  <xacro:property name="base_mass" value="20.0" />
-  <!-- xacro macros -->
+  <!-- gripper instance-->
+  <xacro:vacuum_gripper_definition prefix="${arm_prefix}" gripper_adjustment="0.01"/>
+  <!-- end: compentens instantiating -->
+  <!-- start: xacro cylinder inertial -->
   <xacro:macro name="cylinder_inertial" params="radius length mass *origin">
     <inertial>
@@ -24,28 +32,31 @@
     </inertial>
   </xacro:macro>
+  <!-- end: xacro cylinder inertial -->
+  <!-- start: xacro cylinder geometry -->
   <xacro:macro name="cylinder_geometry" params="radius length">
     <cylinder radius="${radius}" length="${length}"/>
   </xacro:macro>
-  <!-- start: world link -->
+  <!-- end: xacro cylinder geometry -->
+  <!-- start: world link/joint -->
   <link name="world" />
   <joint name="world_to_stand" type="fixed">
     <parent link="world" />
     <child link = "stand_link" />
-    <origin xyz="0.0 0.0 ${base_length/2}" rpy="0.0 0.0 0.0" />
+    <origin xyz="0.0 0.0 ${stand_length/2}" rpy="0.0 0.0 0.0" />
   </joint>
   <!-- end: world link -->
-  <!-- start: base link -->
+  <!-- start: base link/joint -->
   <link name="stand_link">
     <visual>
       <geometry>
-        <xacro:cylinder_geometry radius="${base_radius}" length="${base_length}" />
+        <xacro:cylinder_geometry radius="${stand_radius}" length="${stand_length}" />
       </geometry>
     </visual>
     <collision>
       <geometry>
-        <xacro:cylinder_geometry radius="${base_radius}" length="${base_length}" />
+        <xacro:cylinder_geometry radius="${stand_radius}" length="${stand_length}" />
       </geometry>
     </collision>
-    <xacro:cylinder_inertial radius="${base_radius}" length="${base_length}" mass="${base_mass}">
+    <xacro:cylinder_inertial radius="${stand_radius}" length="${stand_length}" mass="${stand_mass}">
       <origin xyz="0.0 0.0 0.0" rpy="0 0 0" />
     </xacro:cylinder_inertial>
@@ -54,6 +65,34 @@
     <parent link="stand_link" />
     <child link = "base_link" />
-    <origin xyz="0.0 0.0 ${base_length/2}" rpy="0.0 0.0 0.0" />
+    <origin xyz="0.0 0.0 ${stand_length/2}" rpy="0.0 0.0 0.0" />
   </joint>
   <!-- end: base link -->
+  <!-- start: gripper interface plate link/joint -->
+  <link name="${arm_prefix}tool_interface_plate">
+    <visual>
+      <geometry>
+        <box size="0.09525 0.09525 0.0127"/>
+      </geometry>
+      <material name="orange_transparent"/>
+    </visual>
+    <collision>
+      <geometry>
+        <box size="0.09525 0.09525 0.0127"/>
+      </geometry>
+      <material name="blue_transparent"/>
+    </collision>
+  </link>
+  <joint name="${arm_prefix}to_interface_plate" type="fixed">
+    <parent link="${arm_prefix}ee_link"/>
+    <child link="${arm_prefix}tool_interface_plate"/>
+    <origin xyz="0.00635 0 0" rpy="0 1.57  0"/> <!-- 0 1.57 0 -->
+  </joint>
+  <!-- end: gripper interface plate link/joint -->
+  <!-- start: arm-gripper joint -->
+    <joint name="${arm_prefix}to_gripper" type="fixed">
+      <parent link="${arm_prefix}ee_link"/>
+      <child link="${arm_prefix}gripper_frame"/>
+      <origin xyz="0.02 0 0" rpy="-1.57 0 -1.57"/> <!-- 0 1.57 0 -->
+    </joint>
+    <!-- end: arm-gripper joint -->
 </robot>

File: mrk_robot_support/urdf/vacuum_gripper_macro.xacro (robot description, xacro)
@@ -16,5 +16,5 @@
 				<origin xyz="0 0 -0.048" rpy="0 0 0"/>
 				<geometry>
-					<mesh filename="package://robot_config/meshes/vacuum_gripper_single_suction_cup.STL" />
+					<mesh filename="package://mrk_robot_support/meshes/vacuum_gripper_single_suction_cup.STL" />
 				</geometry>
 				<material name="silver">

Commit message: Vacuum gripper mounted correctly

File: mrk_robot_support/urdf/ur5_gripper.xacro (robot description, xacro)
@@ -68,5 +68,5 @@
   </joint>
   <!-- end: base link -->
-  <!-- start: gripper interface plate link/joint -->
+  <!-- start: gripper interface plate link/joint
   <link name="${arm_prefix}tool_interface_plate">
     <visual>
@@ -86,12 +86,12 @@
     <parent link="${arm_prefix}ee_link"/>
     <child link="${arm_prefix}tool_interface_plate"/>
-    <origin xyz="0.00635 0 0" rpy="0 1.57  0"/> <!-- 0 1.57 0 -->
+    <origin xyz="0.00635 0 0" rpy="0 1.57  0"/>
   </joint>
-  <!-- end: gripper interface plate link/joint -->
+  end: gripper interface plate link/joint -->
   <!-- start: arm-gripper joint -->
     <joint name="${arm_prefix}to_gripper" type="fixed">
       <parent link="${arm_prefix}ee_link"/>
       <child link="${arm_prefix}gripper_frame"/>
-      <origin xyz="0.02 0 0" rpy="-1.57 0 -1.57"/> <!-- 0 1.57 0 -->
+      <origin xyz="0 0 0" rpy="-1.57 0 -1.57"/> <!-- 0 1.57 0 -->
     </joint>
     <!-- end: arm-gripper joint -->

Commit message: Vacuum gripper without plate. Visualization in Gazebo working

File: mrk_robot_support/urdf/ur5_gripper.xacro (robot description, xacro)
@@ -1,4 +1,4 @@
 <?xml version="1.0" ?>
-<robot name="ur5_gripper" xmlns:xacro="https://ros.org/wiki/xacro">
+<robot name="ur5_gripper" xmlns:xacro="http://ros.org/wiki/xacro">
   <!-- start: including -->
   <!-- vacum gripper -->
@@ -68,25 +68,4 @@
   </joint>
   <!-- end: base link -->
-  <!-- start: gripper interface plate link/joint
-  <link name="${arm_prefix}tool_interface_plate">
-    <visual>
-      <geometry>
-        <box size="0.09525 0.09525 0.0127"/>
-      </geometry>
-      <material name="orange_transparent"/>
-    </visual>
-    <collision>
-      <geometry>
-        <box size="0.09525 0.09525 0.0127"/>
-      </geometry>
-      <material name="blue_transparent"/>
-    </collision>
-  </link>
-  <joint name="${arm_prefix}to_interface_plate" type="fixed">
-    <parent link="${arm_prefix}ee_link"/>
-    <child link="${arm_prefix}tool_interface_plate"/>
-    <origin xyz="0.00635 0 0" rpy="0 1.57  0"/>
-  </joint>
-  end: gripper interface plate link/joint -->
   <!-- start: arm-gripper joint -->
     <joint name="${arm_prefix}to_gripper" type="fixed">

Commit message: RGB-D sensor added and working. rviz config file added.

File: mrk_robot_support/urdf/ur5_gripper.xacro (robot description, xacro)
@@ -7,8 +7,11 @@
   <xacro:include filename="$(find ur_description)/urdf/common.gazebo.xacro" />
   <xacro:include filename="$(find mrk_robot_support)/urdf/gazebo_extension.xacro" />
+  <!-- RGB-D camera -->
+  <xacro:include filename="$(find mrk_robot_support)/urdf/sensors/xtion_pro_live.urdf.xacro"/>
   <!-- ur5 -->
   <xacro:include filename="$(find ur_description)/urdf/ur5.urdf.xacro" />
   <!-- end: including -->
   <!-- start: properties -->
+  <xacro:property name="deg_to_rad" value="0.01745329251994329577"/>
   <xacro:property name="stand_radius" value="0.08" />
   <xacro:property name="stand_length" value="1.1" />
@@ -20,4 +23,9 @@
   <xacro:ur5_robot prefix="${arm_prefix}" joint_limited="true"/>
   <!-- gripper instance-->
+  <!-- RGB-D camera instance -->
+  <xacro:xtion_pro_live name="rgbd_camera" parent="base">
+    <origin xyz="0.1 0 1" rpy="0 ${75.0 * deg_to_rad} 0"/>
+    <origin xyz="0 0 0" rpy="${-90.0 * deg_to_rad} 0 ${-90.0 * deg_to_rad}"/>
+  </xacro:xtion_pro_live>
   <!-- end: compentens instantiating -->
   <!-- start: xacro cylinder inertial -->

Commit message: set start_tollerance to 0. changed sensor height.

File: mrk_robot_support/urdf/ur5_gripper.xacro (robot description, xacro)
@@ -25,5 +25,5 @@
   <!-- RGB-D camera instance -->
   <xacro:xtion_pro_live name="rgbd_camera" parent="base">
-    <origin xyz="0.1 0 1" rpy="0 ${75.0 * deg_to_rad} 0"/>
+    <origin xyz="0.1 0 2" rpy="0 ${75.0 * deg_to_rad} 0"/>
     <origin xyz="0 0 0" rpy="${-90.0 * deg_to_rad} 0 ${-90.0 * deg_to_rad}"/>
   </xacro:xtion_pro_live>

Commit message: Workbench with collision. RGBD Kamera turned.

File: mrk_robot_support/urdf/ur5_gripper.xacro (robot description, xacro)
@@ -25,5 +25,5 @@
   <!-- RGB-D camera instance -->
   <xacro:xtion_pro_live name="rgbd_camera" parent="base">
-    <origin xyz="0.1 0 2" rpy="0 ${75.0 * deg_to_rad} 0"/>
+    <origin xyz="0.1 0 2" rpy="0 ${75.0 * deg_to_rad} ${-90.0 * deg_to_rad}"/>
     <origin xyz="0 0 0" rpy="${-90.0 * deg_to_rad} 0 ${-90.0 * deg_to_rad}"/>
   </xacro:xtion_pro_live>

Commit message: Object placing improved. Grasping not working.

File: mrk_robot_support/urdf/ur5_gripper.xacro (robot description, xacro)
@@ -15,5 +15,5 @@
   <xacro:property name="deg_to_rad" value="0.01745329251994329577"/>
   <xacro:property name="stand_radius" value="0.08" />
-  <xacro:property name="stand_length" value="1.1" />
+  <xacro:property name="stand_length" value="1.0" />
   <xacro:property name="stand_mass" value="20.0" />
   <xacro:property name="arm_prefix" value=""/>
