Commit message: Splitted launch files.

File: mrk_robot_support/urdf/gripper.xacro (robot description, xacro)
@@ -1,8 +1,13 @@
 <?xml version="1.0" ?>
 <robot name="gripper" xmlns:xacro="http://ros.org/wiki/xacro">
+  <!-- start: Properties -->
   <xacro:property name="pi" value="3.1415926535897931" />
   <xacro:property name="finger_width" value="0.03" />
-  <xacro:property name="finger_length" value="0.2" />
+  <xacro:property name="finger_length" value="0.12" />
+  <xacro:property name="ankle_width" value="0.03" />
+  <xacro:property name="ankle_length" value="0.2" />
   <xacro:property name="mass" value="0.1" />
+  <!-- end: Properties -->
+  <!-- start: Macro Definitions -->
   <xacro:macro name="block" params="name height width depth mass *origin">
     <link name="${name}">
@@ -27,7 +32,11 @@
     </link>
   </xacro:macro>
-  <xacro:block name="gripper_ankle" height="${finger_width}" width="${finger_length}" depth="${finger_width}" mass="${mass}">
+  <!-- end: Macro Definitions -->
+  <!-- start:Gripper Ankle -->
+  <xacro:block name="gripper_ankle" height="${ankle_width}" width="${ankle_length}" depth="${ankle_width}" mass="${mass}">
     <origin xyz="0.0 0.0 ${finger_width/2}" rpy="0 0 ${pi/2}" />
   </xacro:block>
+  <!-- end:Gripper Ankle -->
+  <!-- start: Right Finger -->
   <xacro:block name="gripper_r_finger" height="${finger_width}" width="${finger_length}" depth="${finger_width}" mass="${mass}">
     <origin xyz="${finger_width/2} 0.0 0.0" rpy="0 ${pi/2} 0" />
@@ -40,4 +49,15 @@
     <origin xyz="0.0 0.0 ${finger_length/2 + finger_width}" rpy="${pi/2} 0 ${pi}" />
   </joint>
+  <transmission name="gripper_r_trans">
+    <type>transmission_interface/SimpleTransmission</type>
+    <joint name="r_finger_joint">
+      <hardwareInterface>hardware_interface/EffortJointInterface</hardwareInterface>
+    </joint>
+    <actuator name="gripper_r_motor">
+      <mechanicalReduction>1</mechanicalReduction>
+    </actuator>
+  </transmission>
+  <!-- end: Right Finger -->
+  <!-- start: Left Finger -->
   <xacro:block name="gripper_l_finger" height="${finger_width}" width="${finger_length}" depth="${finger_width}" mass="${mass}">
     <origin xyz="${finger_width/2} 0.0 0.0" rpy="0 0 0" />
@@ -50,13 +70,4 @@
     <origin xyz="0.0 0.0 ${finger_length/2 + finger_width}" rpy="${pi/2} 0 0" />
   </joint>
-  <transmission name="gripper_r_trans">
-    <type>transmission_interface/SimpleTransmission</type>
-    <joint name="r_finger_joint">
-      <hardwareInterface>hardware_interface/EffortJointInterface</hardwareInterface>
-    </joint>
-    <actuator name="gripper_r_motor">
-      <mechanicalReduction>1</mechanicalReduction>
-    </actuator>
-  </transmission>
   <transmission name="gripper_l_trans">
     <type>transmission_interface/SimpleTransmission</type>
@@ -68,3 +79,4 @@
     </actuator>
   </transmission>
+  <!-- end: Left Finger -->
 </robot>

File: mrk_robot_support/urdf/ur5_gripper.xacro (robot description, xacro)
@@ -15,5 +15,5 @@
   <xacro:property name="deg_to_rad" value="0.01745329251994329577"/>
   <xacro:property name="stand_radius" value="0.08" />
-  <xacro:property name="stand_length" value="1.0" />
+  <xacro:property name="stand_length" value="1.2" />
   <xacro:property name="stand_mass" value="20.0" />
   <xacro:property name="arm_prefix" value=""/>

Commit message: Gripper frames changed. Default open.

File: mrk_robot_support/urdf/gripper.xacro (robot description, xacro)
@@ -40,12 +40,12 @@
   <!-- start: Right Finger -->
   <xacro:block name="gripper_r_finger" height="${finger_width}" width="${finger_length}" depth="${finger_width}" mass="${mass}">
-    <origin xyz="${finger_width/2} 0.0 0.0" rpy="0 ${pi/2} 0" />
+    <origin xyz="${finger_width/2} 0.0 0.0" rpy="0 0 0" />
   </xacro:block>
   <joint name="r_finger_joint" type="prismatic">
-    <limit lower="${0}" upper="${finger_length/2 - finger_width}" effort="100.0" velocity="5.0"/>
+    <limit lower="${0}" upper="${ankle_length/2 - finger_width}" effort="100.0" velocity="5.0"/>
     <dynamics damping="0.1"></dynamics>
     <parent link="gripper_ankle"/>
     <child link="gripper_r_finger"/>
-    <origin xyz="0.0 0.0 ${finger_length/2 + finger_width}" rpy="${pi/2} 0 ${pi}" />
+    <origin xyz="${-ankle_length/2} 0.0 ${finger_length/2 + ankle_width}" rpy="${pi/2} 0 0" />
   </joint>
   <transmission name="gripper_r_trans">
@@ -64,9 +64,9 @@
   </xacro:block>
   <joint name="l_finger_joint" type="prismatic">
-    <limit lower="${0}" upper="${finger_length/2 - finger_width}" effort="100.0" velocity="5.0"/>
+    <limit lower="${0}" upper="${ankle_length/2 - finger_width}" effort="100.0" velocity="5.0"/>
     <dynamics damping="0.1"></dynamics>
     <parent link="gripper_ankle"/>
     <child link="gripper_l_finger"/>
-    <origin xyz="0.0 0.0 ${finger_length/2 + finger_width}" rpy="${pi/2} 0 0" />
+    <origin xyz="${ankle_length/2} 0.0 ${finger_length/2 + ankle_width}" rpy="${pi/2} 0 ${pi}" />
   </joint>
   <transmission name="gripper_l_trans">

Commit message: Updated gripper with TCP. Updated moveit config.

File: mrk_robot_support/urdf/gripper.xacro (robot description, xacro)
@@ -80,3 +80,11 @@
   </transmission>
   <!-- end: Left Finger -->
+  <!-- start: Tool Center Point (TCP) -->
+  <link name="tcp_link"/>
+  <joint name="tcp_joint" type="fixed">
+    <origin xyz="0 0 ${ankle_width + finger_length/2}" rpy="0 ${-pi/2} ${-pi/2}"/>
+    <parent link="gripper_ankle"/>
+    <child link="tcp_link"/>
+  </joint>
+  <!-- end: Tool Center Point (TCP) -->
 </robot>

File: mrk_robot_support/urdf/ur5_gripper.xacro (robot description, xacro)
@@ -76,9 +76,9 @@
   <!-- end: base link -->
   <!-- start: arm-gripper joint -->
-    <joint name="${arm_prefix}to_gripper" type="fixed">
-      <parent link="${arm_prefix}ee_link"/>
-      <child link="gripper_ankle"/>
-      <origin xyz="0 0 0" rpy="-1.57 0 -1.57"/>
-    </joint>
+  <joint name="${arm_prefix}to_gripper" type="fixed">
+    <parent link="${arm_prefix}ee_link"/>
+    <child link="gripper_ankle"/>
+    <origin xyz="0 0 0" rpy="-1.57 0 -1.57"/>
+  </joint>
   <!-- end: arm-gripper joint -->
 </robot>

Commit message: Changed gripper link names.

File: mrk_robot_support/urdf/gripper.xacro (robot description, xacro)
@@ -33,11 +33,11 @@
   </xacro:macro>
   <!-- end: Macro Definitions -->
-  <!-- start:Gripper Ankle -->
-  <xacro:block name="gripper_ankle" height="${ankle_width}" width="${ankle_length}" depth="${ankle_width}" mass="${mass}">
+  <!-- start:Gripper Link -->
+  <xacro:block name="gripper_link" height="${ankle_width}" width="${ankle_length}" depth="${ankle_width}" mass="${mass}">
     <origin xyz="0.0 0.0 ${finger_width/2}" rpy="0 0 ${pi/2}" />
   </xacro:block>
-  <!-- end:Gripper Ankle -->
+  <!-- end:Gripper Link -->
   <!-- start: Right Finger -->
-  <xacro:block name="gripper_r_finger" height="${finger_width}" width="${finger_length}" depth="${finger_width}" mass="${mass}">
+  <xacro:block name="r_finger_link" height="${finger_width}" width="${finger_length}" depth="${finger_width}" mass="${mass}">
     <origin xyz="${finger_width/2} 0.0 0.0" rpy="0 0 0" />
   </xacro:block>
@@ -45,14 +45,14 @@
     <limit lower="${0}" upper="${ankle_length/2 - finger_width}" effort="100.0" velocity="5.0"/>
     <dynamics damping="0.1"></dynamics>
-    <parent link="gripper_ankle"/>
-    <child link="gripper_r_finger"/>
+    <parent link="gripper_link"/>
+    <child link="r_finger_link"/>
     <origin xyz="${-ankle_length/2} 0.0 ${finger_length/2 + ankle_width}" rpy="${pi/2} 0 0" />
   </joint>
-  <transmission name="gripper_r_trans">
+  <transmission name="r_finger_trans">
     <type>transmission_interface/SimpleTransmission</type>
     <joint name="r_finger_joint">
       <hardwareInterface>hardware_interface/EffortJointInterface</hardwareInterface>
     </joint>
-    <actuator name="gripper_r_motor">
+    <actuator name="r_finger_motor">
       <mechanicalReduction>1</mechanicalReduction>
     </actuator>
@@ -60,5 +60,5 @@
   <!-- end: Right Finger -->
   <!-- start: Left Finger -->
-  <xacro:block name="gripper_l_finger" height="${finger_width}" width="${finger_length}" depth="${finger_width}" mass="${mass}">
+  <xacro:block name="l_finger_link" height="${finger_width}" width="${finger_length}" depth="${finger_width}" mass="${mass}">
     <origin xyz="${finger_width/2} 0.0 0.0" rpy="0 0 0" />
   </xacro:block>
@@ -66,14 +66,14 @@
     <limit lower="${0}" upper="${ankle_length/2 - finger_width}" effort="100.0" velocity="5.0"/>
     <dynamics damping="0.1"></dynamics>
-    <parent link="gripper_ankle"/>
-    <child link="gripper_l_finger"/>
+    <parent link="gripper_link"/>
+    <child link="l_finger_link"/>
     <origin xyz="${ankle_length/2} 0.0 ${finger_length/2 + ankle_width}" rpy="${pi/2} 0 ${pi}" />
   </joint>
-  <transmission name="gripper_l_trans">
+  <transmission name="l_finger_trans">
     <type>transmission_interface/SimpleTransmission</type>
     <joint name="l_finger_joint">
       <hardwareInterface>hardware_interface/EffortJointInterface</hardwareInterface>
     </joint>
-    <actuator name="gripper_l_motor">
+    <actuator name="l_finger_motor">
       <mechanicalReduction>1</mechanicalReduction>
     </actuator>
@@ -83,6 +83,6 @@
   <link name="tcp_link"/>
   <joint name="tcp_joint" type="fixed">
-    <origin xyz="0 0 ${ankle_width + finger_length/2}" rpy="0 ${-pi/2} ${-pi/2}"/>
-    <parent link="gripper_ankle"/>
+    <origin xyz="0 0 ${ankle_width + finger_length/2}" rpy="0 ${-pi/2} ${pi/2}"/>
+    <parent link="gripper_link"/>
     <child link="tcp_link"/>
   </joint>

File: mrk_robot_support/urdf/ur5_gripper_without_camera.urdf (robot description, URDF)
Before this commit: robot ur5_gripper, 22 links, 21 joints
Links:
- removed link rgbd_camera_depth_frame
- removed link rgbd_camera_depth_optical_frame
- removed link rgbd_camera_link
- removed link rgbd_camera_optical_frame
- removed link rgbd_camera_rgb_frame
- removed link rgbd_camera_rgb_optical_frame
Joints:
- removed joint rgbd_camera_depth_joint
- removed joint rgbd_camera_depth_optical_joint
- removed joint rgbd_camera_joint
- removed joint rgbd_camera_optical_joint
- removed joint rgbd_camera_rgb_joint
- removed joint rgbd_camera_rgb_optical_joint

File: mrk_robot_support/urdf/ur5_gripper_without_camera.xacro (robot description, xacro)
@@ -1,4 +1,4 @@
 <?xml version="1.0" ?>
-<robot name="ur5_gripper" xmlns:xacro="http://ros.org/wiki/xacro">
+<robot name="ur5_gripper_without_camera" xmlns:xacro="http://ros.org/wiki/xacro">
   <!-- start: including -->
   <!-- gripper -->
@@ -8,5 +8,5 @@
   <xacro:include filename="$(find mrk_robot_support)/urdf/gazebo_extension.xacro" />
   <!-- RGB-D camera -->
-  <xacro:include filename="$(find mrk_robot_support)/urdf/sensors/xtion_pro_live.urdf.xacro"/>
+  <!-- <xacro:include filename="$(find mrk_robot_support)/urdf/sensors/xtion_pro_live.urdf.xacro"/> -->
   <!-- ur5 -->
   <xacro:include filename="$(find ur_description)/urdf/ur5.urdf.xacro" />
@@ -19,13 +19,13 @@
   <xacro:property name="arm_prefix" value=""/>
   <!-- end: properties -->
-  <!-- start: compentens instantiating -->
+  <!-- start: compontens instantiating -->
   <!-- arm instance-->
   <xacro:ur5_robot prefix="${arm_prefix}" joint_limited="true"/>
   <!-- gripper instance-->
   <!-- RGB-D camera instance -->
-  <xacro:xtion_pro_live name="rgbd_camera" parent="base">
-    <origin xyz="0.1 0 2" rpy="0 ${75.0 * deg_to_rad} ${-90.0 * deg_to_rad}"/>
-    <origin xyz="0 0 0" rpy="${-90.0 * deg_to_rad} 0 ${-90.0 * deg_to_rad}"/>
-  </xacro:xtion_pro_live>
+  <!-- <xacro:xtion_pro_live name="rgbd_camera" parent="base"> -->
+  <!--   <origin xyz="0.1 0 2" rpy="0 ${75.0 * deg_to_rad} ${-90.0 * deg_to_rad}"/> -->
+  <!--   <origin xyz="0 0 0" rpy="${-90.0 * deg_to_rad} 0 ${-90.0 * deg_to_rad}"/> -->
+  <!-- </xacro:xtion_pro_live> -->
   <!-- end: compentens instantiating -->
   <!-- start: xacro cylinder inertial -->
