Commit message: Simple gripper moving with scripts. Simple beer.world launching

File: mrk_robot_support/urdf/gazebo_extension.xacro (robot description, xacro)
@@ -3,7 +3,17 @@
   <gazebo>
     <plugin name="joint_state_publisher" filename="libgazebo_ros_joint_state_publisher.so">
-      <jointName>shoulder_pan_joint, shoulder_lift_joint, elbow_joint, wrist_1_joint, wrist_2_joint, wrist_3_joint</jointName>
+      <jointName>shoulder_pan_joint, shoulder_lift_joint, elbow_joint, wrist_1_joint, wrist_2_joint, wrist_3_joint, gripper_r_finger_to_ankle</jointName>
       <updateRate>100</updateRate>
     </plugin>
+    <plugin name="gazebo_mimic_plugin" filename="libroboticsgroup_gazebo_mimic_joint_plugin.so">
+      <joint>gripper_r_finger_to_ankle</joint>
+      <mimicJoint>gripper_l_finger_to_ankle</mimicJoint>
+      <multiplier>-1</multiplier>
+    </plugin>
+  </gazebo>
+  <gazebo reference="gripper_r_finger">
+    <mu1>0.2</mu1>
+    <mu2>0.2</mu2>
+    <material>Gazebo/Black</material>
   </gazebo>
 </robot>

File: mrk_robot_support/urdf/ur5_gripper.xacro (robot description, xacro)
@@ -2,6 +2,6 @@
 <robot name="ur5_gripper" xmlns:xacro="http://ros.org/wiki/xacro">
   <!-- start: including -->
-  <!-- vacum gripper -->
-  <xacro:include filename="$(find mrk_robot_support)/urdf/vacuum_gripper_macro.xacro"/>
+  <!-- gripper -->
+  <xacro:include filename="$(find mrk_robot_support)/urdf/gripper.xacro" />
   <!-- gazebo stuff -->
   <xacro:include filename="$(find ur_description)/urdf/common.gazebo.xacro" />
@@ -12,5 +12,5 @@
   <!-- start: properties -->
   <xacro:property name="stand_radius" value="0.08" />
-  <xacro:property name="stand_length" value="0.5" />
+  <xacro:property name="stand_length" value="1.03" />
   <xacro:property name="stand_mass" value="20.0" />
   <xacro:property name="arm_prefix" value=""/>
@@ -18,7 +18,6 @@
   <!-- start: compentens instantiating -->
   <!-- arm instance-->
-  <xacro:ur5_robot prefix="" joint_limited="true"/>
+  <xacro:ur5_robot prefix="${arm_prefix}" joint_limited="true"/>
   <!-- gripper instance-->
-  <xacro:vacuum_gripper_definition prefix="${arm_prefix}" gripper_adjustment="0.01"/>
   <!-- end: compentens instantiating -->
   <!-- start: xacro cylinder inertial -->
@@ -71,7 +70,7 @@
     <joint name="${arm_prefix}to_gripper" type="fixed">
       <parent link="${arm_prefix}ee_link"/>
-      <child link="${arm_prefix}gripper_frame"/>
-      <origin xyz="0 0 0" rpy="-1.57 0 -1.57"/> <!-- 0 1.57 0 -->
+      <child link="gripper_ankle"/>
+      <origin xyz="0 0 0" rpy="-1.57 0 -1.57"/>
     </joint>
-    <!-- end: arm-gripper joint -->
+  <!-- end: arm-gripper joint -->
 </robot>

Commit message: Gripper beer grasping in Gazebo. Wait for a few seconds for grasping.

File: mrk_robot_support/urdf/gazebo_extension.xacro (robot description, xacro)
@@ -3,17 +3,34 @@
   <gazebo>
     <plugin name="joint_state_publisher" filename="libgazebo_ros_joint_state_publisher.so">
-      <jointName>shoulder_pan_joint, shoulder_lift_joint, elbow_joint, wrist_1_joint, wrist_2_joint, wrist_3_joint, gripper_r_finger_to_ankle</jointName>
+      <jointName>shoulder_pan_joint, shoulder_lift_joint, elbow_joint, wrist_1_joint, wrist_2_joint, wrist_3_joint, r_finger_joint, l_finger_joint</jointName>
       <updateRate>100</updateRate>
     </plugin>
-    <plugin name="gazebo_mimic_plugin" filename="libroboticsgroup_gazebo_mimic_joint_plugin.so">
-      <joint>gripper_r_finger_to_ankle</joint>
-      <mimicJoint>gripper_l_finger_to_ankle</mimicJoint>
-      <multiplier>-1</multiplier>
-    </plugin>
+    <!-- <plugin name="gazebo_mimic_plugin" filename="libroboticsgroup_gazebo_mimic_joint_plugin.so"> -->
+    <!--   <joint>r_finger_joint</joint> -->
+    <!--   <mimicJoint>l_finger_joint</mimicJoint> -->
+    <!--   <multiplier>-1</multiplier> -->
+    <!-- </plugin> -->
   </gazebo>
   <gazebo reference="gripper_r_finger">
-    <mu1>0.2</mu1>
-    <mu2>0.2</mu2>
-    <material>Gazebo/Black</material>
+    <mu1>100</mu1>
+    <mu2>100</mu2>
+    <material>Gazebo/Blue</material>
+  </gazebo>
+  <gazebo reference="gripper_l_finger">
+    <mu1>100</mu1>
+    <mu2>100</mu2>
+    <material>Gazebo/Red</material>
+  </gazebo>
+  <gazebo>
+    <gripper name="grasping">
+        <grasp_check>
+            <attach_steps>3</attach_steps>
+            <detach_steps>3</detach_steps>
+            <min_contact_count>1</min_contact_count>
+        </grasp_check>
+        <gripper_link>gripper_r_finger</gripper_link>
+        <gripper_link>gripper_l_finger</gripper_link>
+        <palm_link>gripper_ankle</palm_link>
+    </gripper>
   </gazebo>
 </robot>

File: mrk_robot_support/urdf/gripper.xacro (robot description, xacro)
@@ -31,30 +31,40 @@
   </xacro:block>
   <xacro:block name="gripper_r_finger" height="${finger_width}" width="${finger_length}" depth="${finger_width}" mass="${mass}">
-    <origin xyz="0.0 0.0 0.0" rpy="0 ${pi/2} 0" />
+    <origin xyz="${finger_width/2} 0.0 0.0" rpy="0 ${pi/2} 0" />
   </xacro:block>
-  <joint name="gripper_r_finger_to_ankle" type="prismatic">
-    <limit lower="${finger_width/2}" upper="${finger_length/2 - finger_width/2}" effort="100" velocity="0.25"/>
+  <joint name="r_finger_joint" type="prismatic">
+    <limit lower="${0}" upper="${finger_length/2 - finger_width}" effort="100" velocity="0.25"/>
     <dynamics damping="0.1"></dynamics>
     <parent link="gripper_ankle"/>
     <child link="gripper_r_finger"/>
-    <origin xyz="0.0 0.0 ${finger_length/2 + finger_width}" rpy="${pi/2} 0 0" />
+    <origin xyz="0.0 0.0 ${finger_length/2 + finger_width}" rpy="${pi/2} 0 ${pi}" />
   </joint>
   <xacro:block name="gripper_l_finger" height="${finger_width}" width="${finger_length}" depth="${finger_width}" mass="${mass}">
-    <origin xyz="0.0 0.0 0.0" rpy="0 0 0" />
+    <origin xyz="${finger_width/2} 0.0 0.0" rpy="0 0 0" />
   </xacro:block>
-  <joint name="gripper_l_finger_to_ankle" type="prismatic">
-    <limit lower="-${finger_width/2}" upper="-${finger_length/2 - finger_width/2}" effort="100" velocity="0.25"/>
+  <joint name="l_finger_joint" type="prismatic">
+    <limit lower="${0}" upper="${finger_length/2 - finger_width}" effort="100" velocity="0.25"/>
     <dynamics damping="0.1"></dynamics>
-    <mimic joint="gripper_r_finger_to_ankle" multiplier="-1" />
     <parent link="gripper_ankle"/>
     <child link="gripper_l_finger"/>
     <origin xyz="0.0 0.0 ${finger_length/2 + finger_width}" rpy="${pi/2} 0 0" />
   </joint>
-  <transmission name="gripper_trans">
+  <transmission name="gripper_r_trans">
     <type>transmission_interface/SimpleTransmission</type>
-    <joint name="gripper_r_finger_to_ankle">
-      <hardwareInterface>hardware_interface/PositionJointInterface</hardwareInterface>
+    <joint name="r_finger_joint">
+      <hardwareInterface>hardware_interface/EffortJointInterface</hardwareInterface>
     </joint>
-    <actuator name="gripper_motor" />
+    <actuator name="gripper_r_motor">
+      <mechanicalReduction>1</mechanicalReduction>
+    </actuator>
+  </transmission>
+  <transmission name="gripper_l_trans">
+    <type>transmission_interface/SimpleTransmission</type>
+    <joint name="l_finger_joint">
+      <hardwareInterface>hardware_interface/EffortJointInterface</hardwareInterface>
+    </joint>
+    <actuator name="gripper_l_motor">
+      <mechanicalReduction>1</mechanicalReduction>
+    </actuator>
   </transmission>
 </robot>

File: mrk_robot_support/urdf/ur5_gripper.xacro (robot description, xacro)
@@ -12,5 +12,5 @@
   <!-- start: properties -->
   <xacro:property name="stand_radius" value="0.08" />
-  <xacro:property name="stand_length" value="1.03" />
+  <xacro:property name="stand_length" value="1.1" />
   <xacro:property name="stand_mass" value="20.0" />
   <xacro:property name="arm_prefix" value=""/>

Commit message: moveit tests. moveit_commander not working

File: mrk_robot_support/urdf/gazebo_extension.xacro (robot description, xacro)
@@ -13,11 +13,11 @@
   </gazebo>
   <gazebo reference="gripper_r_finger">
-    <mu1>0.9</mu1>
-    <mu2>0.9</mu2>
-    <material>Gazebo/Blue</material>
+    <mu1>0.2</mu1>
+    <mu2>0.2</mu2>
+   <material>Gazebo/Blue</material>
   </gazebo>
   <gazebo reference="gripper_l_finger">
-    <mu1>0.9</mu1>
-    <mu2>0.9</mu2>
+    <mu1>0.2</mu1>
+    <mu2>0.2</mu2>
     <material>Gazebo/Red</material>
   </gazebo>
@@ -26,5 +26,5 @@
         <grasp_check>
             <attach_steps>3</attach_steps>
-            <detach_steps>10</detach_steps>
+            <detach_steps>3</detach_steps>
             <min_contact_count>1</min_contact_count>
         </grasp_check>

File: mrk_robot_support/urdf/gripper.xacro (robot description, xacro)
@@ -34,5 +34,5 @@
   </xacro:block>
   <joint name="r_finger_joint" type="prismatic">
-    <limit lower="${0}" upper="${finger_length/2 - finger_width}" effort="100" velocity="0.25"/>
+    <limit lower="${0}" upper="${finger_length/2 - finger_width}" effort="100.0" velocity="5.0"/>
     <dynamics damping="0.1"></dynamics>
     <parent link="gripper_ankle"/>
@@ -44,5 +44,5 @@
   </xacro:block>
   <joint name="l_finger_joint" type="prismatic">
-    <limit lower="${0}" upper="${finger_length/2 - finger_width}" effort="100" velocity="0.25"/>
+    <limit lower="${0}" upper="${finger_length/2 - finger_width}" effort="100.0" velocity="5.0"/>
     <dynamics damping="0.1"></dynamics>
     <parent link="gripper_ankle"/>

Commit message: Grasp server working

File: mrk_robot_support/urdf/gazebo_extension.xacro (robot description, xacro)
@@ -4,5 +4,5 @@
     <plugin name="joint_state_publisher" filename="libgazebo_ros_joint_state_publisher.so">
       <jointName>shoulder_pan_joint, shoulder_lift_joint, elbow_joint, wrist_1_joint, wrist_2_joint, wrist_3_joint, r_finger_joint, l_finger_joint</jointName>
-      <updateRate>50</updateRate>
+      <updateRate>100</updateRate>
     </plugin>
     <!-- <plugin name="gazebo_mimic_plugin" filename="libroboticsgroup_gazebo_mimic_joint_plugin.so"> -->
@@ -12,25 +12,25 @@
     <!-- </plugin> -->
   </gazebo>
-  <gazebo reference="gripper_r_finger">
-    <mu1>0.2</mu1>
-    <mu2>0.2</mu2>
-   <material>Gazebo/Blue</material>
-  </gazebo>
-  <gazebo reference="gripper_l_finger">
-    <mu1>0.2</mu1>
-    <mu2>0.2</mu2>
-    <material>Gazebo/Red</material>
-  </gazebo>
-  <gazebo>
-    <gripper name="grasping">
-        <grasp_check>
-            <attach_steps>3</attach_steps>
-            <detach_steps>3</detach_steps>
-            <min_contact_count>1</min_contact_count>
-        </grasp_check>
-        <gripper_link>gripper_r_finger</gripper_link>
-        <gripper_link>gripper_l_finger</gripper_link>
-        <palm_link>gripper_ankle</palm_link>
-    </gripper>
-  </gazebo>
+  <!-- <gazebo reference="gripper_r_finger"> -->
+  <!--   <mu1>0.2</mu1> -->
+  <!--   <mu2>0.2</mu2> -->
+  <!--  <material>Gazebo/Blue</material> -->
+  <!-- </gazebo> -->
+  <!-- <gazebo reference="gripper_l_finger"> -->
+  <!--   <mu1>0.2</mu1> -->
+  <!--   <mu2>0.2</mu2> -->
+  <!--   <material>Gazebo/Red</material> -->
+  <!-- </gazebo> -->
+  <!-- <gazebo> -->
+  <!--   <gripper name="grasping"> -->
+  <!--       <grasp_check> -->
+  <!--           <attach_steps>3</attach_steps> -->
+  <!--           <detach_steps>3</detach_steps> -->
+  <!--           <min_contact_count>1</min_contact_count> -->
+  <!--       </grasp_check> -->
+  <!--       <gripper_link>gripper_r_finger</gripper_link> -->
+  <!--       <gripper_link>gripper_l_finger</gripper_link> -->
+  <!--       <palm_link>gripper_ankle</palm_link> -->
+  <!--   </gripper> -->
+  <!-- </gazebo> -->
 </robot>

Commit message: Scrips added. Changed open/closeGripper.sh. Models changed.

File: mrk_robot_support/urdf/gazebo_extension.xacro (robot description, xacro)
@@ -12,14 +12,12 @@
     <!-- </plugin> -->
   </gazebo>
-  <!-- <gazebo reference="gripper_r_finger"> -->
-  <!--   <mu1>0.2</mu1> -->
-  <!--   <mu2>0.2</mu2> -->
-  <!--  <material>Gazebo/Blue</material> -->
-  <!-- </gazebo> -->
-  <!-- <gazebo reference="gripper_l_finger"> -->
-  <!--   <mu1>0.2</mu1> -->
-  <!--   <mu2>0.2</mu2> -->
-  <!--   <material>Gazebo/Red</material> -->
-  <!-- </gazebo> -->
+  <gazebo reference="r_finger_link">
+    <mu1>10</mu1>
+    <mu2>20</mu2>
+  </gazebo>
+  <gazebo reference="l_finger_link">
+    <mu1>10</mu1>
+    <mu2>20</mu2>
+  </gazebo>
   <!-- <gazebo> -->
   <!--   <gripper name="grasping"> -->

File: mrk_robot_support/urdf/gripper.xacro (robot description, xacro)
@@ -88,3 +88,14 @@
   </joint>
   <!-- end: Tool Center Point (TCP) -->
+  <!-- start: Gazebo material information -->
+  <gazebo reference="gripper_link">
+    <material>Gazebo/Orange</material>
+  </gazebo>
+  <gazebo reference="l_finger_link">
+    <material>Gazebo/Orange</material>
+  </gazebo>
+  <gazebo reference="r_finger_link">
+    <material>Gazebo/Orange</material>
+  </gazebo>
+  <!-- end: Gazebo material information -->
 </robot>

File: mrk_robot_support/urdf/ur5_gripper.xacro (robot description, xacro)
@@ -25,5 +25,5 @@
   <!-- RGB-D camera instance -->
   <xacro:xtion_pro_live name="rgbd_camera" parent="base">
-    <origin xyz="0.1 0 2" rpy="0 ${75.0 * deg_to_rad} ${-90.0 * deg_to_rad}"/>
+    <origin xyz="0 0 2" rpy="0 ${75.0 * deg_to_rad} ${-90.0 * deg_to_rad}"/>
     <origin xyz="0 0 0" rpy="${-90.0 * deg_to_rad} 0 ${-90.0 * deg_to_rad}"/>
   </xacro:xtion_pro_live>
@@ -82,3 +82,8 @@
   </joint>
   <!-- end: arm-gripper joint -->
+  <!-- start: Gazebo material information -->
+    <gazebo reference="stand_link">
+      <material>Gazebo/Grey</material>
+    </gazebo>
+  <!-- end: Gazebo material information -->
 </robot>
